File: PcbDesignes/ServoBrushed/combined/combined.sch (KiCad schematic (older format))
At the start: 24 parts, among them M1 Motor_DC, U1 ITR8307, U2 ITR8307, U3 AP2112K-3.3, U4 ATSAMD21G18A-A, U5 TB6612FNG

Commit message: updated version of ServoBrushed combined pcb
Parts:
- D1: footprint Diode_SMD:D_0402_1005Metric -> LED_SMD:LED_0805_2012Metric_Castellated; LCSC C130719 -> C84256
Connections:
- net labels added: USB_D+, USB_D-
Changed lines of the file:
@@
-$EndComp
-$Comp
-L Device:LED D1
-U 1 1 60E9B8ED
-P 3400 5150
-F 0 "D1" H 3393 5367 50  0000 C CNN
-F 1 "LED" H 3393 5276 50  0000 C CNN
-F 2 "Diode_SMD:D_0402_1005Metric" H 3400 5150 50  0001 C CNN
-F 3 "~" H 3400 5150 50  0001 C CNN
-F 4 "C130719 " H 3400 5150 50  0001 C CNN "LCSC"
-	1    3400 5150
-	1    0    0    -1
 $EndComp
 $Comp
@@
 Wire Wire Line
 	3250 5150 3150 5150
+Text Label 1800 5950 0    50   ~ 0
+USB_D+
+Text Label 1800 5850 0    50   ~ 0
+USB_D-
+$Comp
+L Device:LED D1
+U 1 1 60E9B8ED
+P 3400 5150
+F 0 "D1" H 3393 5367 50  0000 C CNN
+F 1 "LED" H 3393 5276 50  0000 C CNN
+F 2 "LED_SMD:LED_0805_2012Metric_Castellated" H 3400 5150 50  0001 C CNN
+F 3 "~" H 3400 5150 50  0001 C CNN
+F 4 "C84256" H 3400 5150 50  0001 C CNN "LCSC"
+	1    3400 5150
+	1    0    0    -1
+$EndComp
 $EndSCHEMATC
